File: hardware/SmartMatrixShield_V1.brd (EAGLE design)
At the start: 48.5 x 36.8 mm, 10 parts, among them J1 CON_HEADER_2X08-PTH-SHROUDED, J4 1X2-5.0

Commit message: Schematic cleanup: Added some clarifying text
Parts:
- renumbered U$1 to U1
Changed lines of the file:
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@@
 <element name="JP2" library="eclibrary" package="1X04-1.56&quot;" value="" x="16.51" y="26.797" smashed="yes"/>
 <element name="D1" library="eclibrary" package="DIODE-TH-0.3&quot;" value="1N400X" x="26.289" y="30.607" smashed="yes" rot="R90"/>
-<element name="U$1" library="eclibrary" package="TEENSY_3.0_MIN" value="TEENSY_3.0_MIN" x="30.48" y="15.24" smashed="yes" rot="R270"/>
+<element name="U1" library="eclibrary" package="TEENSY_3.0_MIN" value="TEENSY_3.0_MIN" x="30.48" y="15.24" smashed="yes" rot="R270"/>
 <element name="JP5" library="eclibrary" package="STAND-OFF-3MM" value="STAND-OFFSTAND-OFF-3MM" x="3.81" y="33.02"/>
 <element name="JP1" library="pinhead-2" package="1X15-S" value="" x="28.702" y="3.175" smashed="yes" rot="R180">
@@
 <signal name="VIN" class="1">
 <contactref element="D1" pad="C"/>
-<contactref element="U$1" pad="VIN"/>
-<contactref element="U$1" pad="VIN"/>
+<contactref element="U1" pad="VIN"/>
+<contactref element="U1" pad="VIN"/>
 <contactref element="JP1" pad="2"/>
 <wire x1="43.942" y1="3.175" x2="43.942" y2="4.572" width="0.508" layer="16"/>
@@
 <signal name="VEXT" class="1">
 <contactref element="CN1" pad="PWR"/>
-<contactref element="D1" pad="A"/>
 <polygon width="0.4064" layer="1" isolate="0.3048">
 <vertex x="16.51" y="36.576"/>
@@
 <wire x1="35.306" y1="28.956" x2="35.803" y2="28.956" width="0.508" layer="1"/>
 <wire x1="35.803" y1="28.956" x2="35.549" y2="29.21" width="0.508" layer="1"/>
+<contactref element="D1" pad="A"/>
+<wire x1="19.01" y1="32.512" x2="26.289" y2="34.417" width="0" layer="19" extent="1-1"/>
+<wire x1="18.4912" y1="26.797" x2="19.01" y2="32.512" width="0" layer="19" extent="1-1"/>
+<wire x1="22.4536" y1="26.797" x2="18.4912" y2="26.797" width="0" layer="19" extent="1-1"/>
+<wire x1="35.306" y1="28.956" x2="26.289" y2="34.417" width="0" layer="19" extent="1-1"/>
 </signal>
 <signal name="GND" class="1">
@@
 <contactref element="J1" pad="8"/>
 <contactref element="J1" pad="16"/>
-<contactref element="U$1" pad="GND"/>
+<contactref element="U1" pad="GND"/>
 <polygon width="0.4064" layer="16" isolate="0.3048">
 <vertex x="48.26" y="36.83"/>
@@
 <signal name="R1">
 <contactref element="J1" pad="1"/>
-<contactref element="U$1" pad="2"/>
+<contactref element="U1" pad="2"/>
 <wire x1="39.37" y1="22.86" x2="37.338" y2="25.019" width="0.254" layer="1"/>
 <wire x1="3.175" y1="22.86" x2="5.207" y2="25.019" width="0.254" layer="1"/>
@@
 <signal name="B1">
 <contactref element="J1" pad="3"/>
-<contactref element="U$1" pad="6"/>
+<contactref element="U1" pad="6"/>
 <wire x1="29.21" y1="22.86" x2="28.194" y2="24.003" width="0.254" layer="1"/>
 <wire x1="28.194" y1="24.003" x2="13.335" y2="24.003" width="0.254" layer="1"/>
@@
 <signal name="R2">
 <contactref element="J1" pad="5"/>
-<contactref element="U$1" pad="21/A7"/>
+<contactref element="U1" pad="21/A7"/>
 <wire x1="3.175" y1="17.78" x2="3.556" y2="17.78" width="0.254" layer="1"/>
 <wire x1="3.556" y1="17.78" x2="4.826" y2="16.51" width="0.254" layer="1"/>
@@
 <signal name="B2">
 <contactref element="J1" pad="7"/>
-<contactref element="U$1" pad="20/A6"/>
+<contactref element="U1" pad="20/A6"/>
 <wire x1="31.75" y1="7.62" x2="29.337" y2="10.287" width="0.254" layer="1"/>
 <wire x1="3.175" y1="15.24" x2="3.175" y2="15.113" width="0.254" layer="1"/>
@@
 <signal name="ADX0">
 <contactref element="J1" pad="9"/>
-<contactref element="U$1" pad="9"/>
+<contactref element="U1" pad="9"/>
 <wire x1="3.175" y1="12.7" x2="1.778" y2="14.097" width="0.254" layer="1"/>
 <wire x1="1.778" y1="14.097" x2="1.778" y2="18.288" width="0.254" layer="1"/>
@@
 <signal name="ADX2">
 <contactref element="J1" pad="11"/>
-<contactref element="U$1" pad="22/A8"/>
+<contactref element="U1" pad="22/A8"/>
 <wire x1="36.83" y1="7.62" x2="35.56" y2="6.35" width="0.254" layer="1"/>
 <wire x1="35.56" y1="6.35" x2="31.242" y2="6.35" width="0.254" layer="1"/>
@@
 <signal name="OE">
 <contactref element="J1" pad="15"/>
-<contactref element="U$1" pad="4"/>
+<contactref element="U1" pad="4"/>
 <via x="11.938" y="8.128" extent="1-16" drill="0.3048"/>
 <via x="12.954" y="20.32" extent="1-16" drill="0.3048"/>
@@
 <signal name="G1">
 <contactref element="J1" pad="2"/>
-<contactref element="U$1" pad="5"/>
+<contactref element="U1" pad="5"/>
 <wire x1="5.715" y1="22.86" x2="5.969" y2="22.606" width="0.254" layer="1"/>
 <wire x1="5.969" y1="22.606" x2="11.43" y2="22.606" width="0.254" layer="1"/>
@@
 <contactref element="J1" pad="6"/>
 <wire x1="5.715" y1="17.78" x2="26.924" y2="17.78" width="0.254" layer="1"/>
-<contactref element="U$1" pad="7"/>
+<contactref element="U1" pad="7"/>
 <wire x1="26.924" y1="17.78" x2="27.686" y2="18.542" width="0.254" layer="1"/>
 <via x="27.686" y="18.542" extent="1-16" drill="0.3048"/>
@@
 <signal name="ADX1">
 <contactref element="J1" pad="10"/>
-<contactref element="U$1" pad="10"/>
+<contactref element="U1" pad="10"/>
 <via x="19.812" y="11.684" extent="1-16" drill="0.3048"/>
 <wire x1="19.05" y1="22.86" x2="18.288" y2="22.098" width="0.254" layer="16"/>
@@
 <signal name="LATCH">
 <contactref element="J1" pad="14"/>
-<contactref element="U$1" pad="3"/>
-<contactref element="U$1" pad="8"/>
+<contactref element="U1" pad="3"/>
+<contactref element="U1" pad="8"/>
 <wire x1="5.715" y1="7.62" x2="8.763" y2="7.62" width="0.254" layer="1"/>
 <wire x1="8.763" y1="7.62" x2="9.271" y2="8.128" width="0.254" layer="1"/>
@@
 <signal name="CLK">
 <contactref element="J1" pad="13"/>
-<contactref element="U$1" pad="14/A0"/>
+<contactref element="U1" pad="14/A0"/>
 <wire x1="16.51" y1="7.62" x2="15.24" y2="8.89" width="0.254" layer="1"/>
 <wire x1="15.24" y1="8.89" x2="4.572" y2="8.89" width="0.254" layer="1"/>
@@
 <signal name="ADX3">
 <contactref element="J1" pad="12"/>
-<contactref element="U$1" pad="23/A9"/>
+<contactref element="U1" pad="23/A9"/>
 <wire x1="39.37" y1="7.62" x2="37.592" y2="5.842" width="0.254" layer="1"/>
 <wire x1="37.592" y1="5.842" x2="29.21" y2="5.842" width="0.254" layer="1"/>
@@
 <contactref element="R1" pad="2"/>
 <contactref element="R2" pad="2"/>
-<contactref element="U$1" pad="3.3V"/>
+<contactref element="U1" pad="3.3V"/>
 <contactref element="JP1" pad="5"/>
 <wire x1="10.795" y1="16.129" x2="10.795" y2="14.478" width="0.4064" layer="1"/>
@@
 <signal name="17/SDA">
 <contactref element="R1" pad="1"/>
-<contactref element="U$1" pad="17/A3"/>
+<contactref element="U1" pad="17/A3"/>
 <contactref element="JP1" pad="10"/>
 <wire x1="23.622" y1="3.175" x2="23.622" y2="7.112" width="0.254" layer="1"/>
@@
 <signal name="16/SCL">
 <contactref element="R2" pad="1"/>
-<contactref element="U$1" pad="16/A2"/>
+<contactref element="U1" pad="16/A2"/>
 <contactref element="JP1" pad="11"/>
 <wire x1="21.082" y1="3.175" x2="21.082" y2="7.112" width="0.254" layer="1"/>
@@
 </signal>
 <signal name="1/UART_TX">
-<contactref element="U$1" pad="1"/>
+<contactref element="U1" pad="1"/>
 <contactref element="JP1" pad="7"/>
 <wire x1="31.242" y1="3.175" x2="33.02" y2="4.953" width="0.254" layer="16"/>
@@
 </signal>
 <signal name="0/UART_RX">
-<contactref element="U$1" pad="0"/>
+<contactref element="U1" pad="0"/>
 <contactref element="JP1" pad="6"/>
 <wire x1="33.782" y1="3.175" x2="35.433" y2="5.334" width="0.254" layer="1"/>
@@
 </signal>
 <signal name="AGND" class="1">
-<contactref element="U$1" pad="AGND"/>
-<contactref element="U$1" pad="AGND"/>
+<contactref element="U1" pad="AGND"/>
+<contactref element="U1" pad="AGND"/>
 <contactref element="JP1" pad="3"/>
 <wire x1="41.402" y1="3.175" x2="41.402" y2="4.572" width="0.508" layer="16"/>
@@
 </signal>
 <signal name="19/UART_RTS">
-<contactref element="U$1" pad="19/A5"/>
+<contactref element="U1" pad="19/A5"/>
 <contactref element="JP1" pad="8"/>
 <wire x1="28.702" y1="3.175" x2="28.702" y2="7.112" width="0.254" layer="16"/>
@@
 </signal>
 <signal name="15/SPI_CS">
-<contactref element="U$1" pad="15/A1"/>
+<contactref element="U1" pad="15/A1"/>
 <contactref element="JP1" pad="12"/>
 <wire x1="18.796" y1="7.366" x2="18.796" y2="3.429" width="0.254" layer="1"/>
@@
 </signal>
 <signal name="13/LED/SPI_SCK">
-<contactref element="U$1" pad="13"/>
+<contactref element="U1" pad="13"/>
 <contactref element="JP1" pad="13"/>
 <wire x1="13.97" y1="7.62" x2="16.002" y2="5.588" width="0.254" layer="1"/>
@@
 </signal>
 <signal name="12/SPI_SIN">
-<contactref element="U$1" pad="12"/>
+<contactref element="U1" pad="12"/>
 <contactref element="JP1" pad="14"/>
 <wire x1="13.97" y1="22.86" x2="13.97" y2="9.652" width="0.254" layer="16"/>
@@
 </signal>
 <signal name="11/SPI_SOUT">
-<contactref element="U$1" pad="11"/>
+<contactref element="U1" pad="11"/>
 <contactref element="JP1" pad="15"/>
 <wire x1="10.922" y1="3.175" x2="12.192" y2="1.905" width="0.254" layer="16"/>
@@
 </signal>
 <signal name="18/UART_CTS">
-<contactref element="U$1" pad="18/A4"/>
+<contactref element="U1" pad="18/A4"/>
 <contactref element="JP1" pad="9"/>
 <wire x1="26.162" y1="3.175" x2="26.162" y2="7.112" width="0.254" layer="1"/>
