File: hardware/SmartMatrixSD_V1.brd (EAGLE design)
At the start: 48.5 x 36.8 mm, 18 parts, among them J1 CON_HEADER_2X08-PTH-SHROUDED, J4 1X2-5.0

Commit message: Remove logo from SmartMatrix SD V1 board files
Parts:
- removed U$5: (no value), eclibrary:PIXELMATIX-LOGO-235X135
Changed lines of the file:
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@@
 <attribute name="VALUE" x="14.986" y="33.909" size="1.27" layer="27" rot="R180"/>
 </element>
-<element name="U$5" library="eclibrary" package="PIXELMATIX-LOGO-235X135" value="" x="47.244" y="11.811" rot="MR0"/>
 <element name="U$3" library="eclibrary" package="TEENSY_3.0_ALLPINS-VUSB-A11-A10-AREF" value="TEENSY_3.0_ALL-VUSB-A10-A11-AREF" x="30.48" y="15.24" smashed="yes" rot="R270"/>
 </elements>
